File: e-ink kb.kicad_sch (KiCad schematic)
At the start: 1 part, among them J1 Conn_01x24_MountingPin

Commit message: finished schematic i think
also added some 3d models, but it is kinda colorless and only on the 1u keys currently.
to-do: pcb part/footprint placements
Parts:
- added C1: 1uF, Capacitor_SMD:C_0805_2012Metric_Pad1.18x1.45mm_HandSolder, symbol Device:C_Small
- added C10, C11, C12, C4, C7, C8, C9: 1uF, Capacitor_SMD:C_0805_2012Metric_Pad1.18x1.45mm_HandSolder, symbol Device:C
- added C13, C14: 2.2uF, Capacitor_SMD:C_0805_2012Metric_Pad1.18x1.45mm_HandSolder, symbol Device:C_Small
- added C15, C16, C17, C18: .1uF, Capacitor_SMD:C_0805_2012Metric_Pad1.18x1.45mm_HandSolder, symbol Device:C_Small
- added C19: .1uF, Capacitor_SMD:C_0805_2012Metric_Pad1.18x1.45mm_HandSolder, symbol Device:C
- added C2, C5, C6: 4.7uF, Capacitor_SMD:C_0805_2012Metric_Pad1.18x1.45mm_HandSolder, symbol Device:C
- added C20: 2.2uF, Capacitor_SMD:C_0805_2012Metric_Pad1.18x1.45mm_HandSolder, symbol Device:C
- added C21, C22: 15pF, Capacitor_SMD:C_0805_2012Metric_Pad1.18x1.45mm_HandSolder, symbol Device:C
- added C3: 10uF, Capacitor_SMD:C_0805_2012Metric_Pad1.18x1.45mm_HandSolder, symbol Device:C
- added D1, D10, D11, D12, D13, D14, D15, D16, D17, D18, D19, D2, D20, D21, D22, D23, D24, D25, D26, D27, D28, D29, D3, D30, D31, D32, D33, D34, D35, D36, D37, D38, D39, D4, D40, D41, D42, D43, D44, D45, D46, D47, D48, D49, D5, D50, D51, D52, D53, D54, D55, D56, D57, D58, D59, D6, D60, D61, D62, D63, D64, D65, D66, D67, D68, D69, D7, D70, D71, D72, D73, D74, D75, D76, D77, D78, D79, D8, D80, D81, D82, D83, D84, D85, D86, D87, D9: D_Small, Diode_SMD:D_SOD-323F, symbol Device:D_Small
- added D100, D98, D99: MBR0530, Diode_SMD:D_SOD-123, symbol Diode:MBR0530
- added D101: ESC, LED_SMD:LED_SK6812MINI-E_3.2x2.8mm_P1.5mm_ReverseMount, symbol LED:SK6812MINI-E
- added D102: F1, LED_SMD:LED_SK6812MINI-E_3.2x2.8mm_P1.5mm_ReverseMount, symbol LED:SK6812MINI-E
- added D103: F2, LED_SMD:LED_SK6812MINI-E_3.2x2.8mm_P1.5mm_ReverseMount, symbol LED:SK6812MINI-E
- added D104: F3, LED_SMD:LED_SK6812MINI-E_3.2x2.8mm_P1.5mm_ReverseMount, symbol LED:SK6812MINI-E
- added D105: F4, LED_SMD:LED_SK6812MINI-E_3.2x2.8mm_P1.5mm_ReverseMount, symbol LED:SK6812MINI-E
- added D106: F5, LED_SMD:LED_SK6812MINI-E_3.2x2.8mm_P1.5mm_ReverseMount, symbol LED:SK6812MINI-E
- added D107: F6, LED_SMD:LED_SK6812MINI-E_3.2x2.8mm_P1.5mm_ReverseMount, symbol LED:SK6812MINI-E
- added D108: F7, LED_SMD:LED_SK6812MINI-E_3.2x2.8mm_P1.5mm_ReverseMount, symbol LED:SK6812MINI-E
- added D109: F8, LED_SMD:LED_SK6812MINI-E_3.2x2.8mm_P1.5mm_ReverseMount, symbol LED:SK6812MINI-E
- added D110: F9, LED_SMD:LED_SK6812MINI-E_3.2x2.8mm_P1.5mm_ReverseMount, symbol LED:SK6812MINI-E
- added D111: F10, LED_SMD:LED_SK6812MINI-E_3.2x2.8mm_P1.5mm_ReverseMount, symbol LED:SK6812MINI-E
- added D112: F11, LED_SMD:LED_SK6812MINI-E_3.2x2.8mm_P1.5mm_ReverseMount, symbol LED:SK6812MINI-E
- added D113: F12, LED_SMD:LED_SK6812MINI-E_3.2x2.8mm_P1.5mm_ReverseMount, symbol LED:SK6812MINI-E
- added D114: PRINT, LED_SMD:LED_SK6812MINI-E_3.2x2.8mm_P1.5mm_ReverseMount, symbol LED:SK6812MINI-E
- added D115: PAUSE, LED_SMD:LED_SK6812MINI-E_3.2x2.8mm_P1.5mm_ReverseMount, symbol LED:SK6812MINI-E
- added D116: SCR LOCK, LED_SMD:LED_SK6812MINI-E_3.2x2.8mm_P1.5mm_ReverseMount, symbol LED:SK6812MINI-E
- added D117: `, LED_SMD:LED_SK6812MINI-E_3.2x2.8mm_P1.5mm_ReverseMount, symbol LED:SK6812MINI-E
- added D118: 1, LED_SMD:LED_SK6812MINI-E_3.2x2.8mm_P1.5mm_ReverseMount, symbol LED:SK6812MINI-E
- added D119: 2, LED_SMD:LED_SK6812MINI-E_3.2x2.8mm_P1.5mm_ReverseMount, symbol LED:SK6812MINI-E
- added D120: 3, LED_SMD:LED_SK6812MINI-E_3.2x2.8mm_P1.5mm_ReverseMount, symbol LED:SK6812MINI-E
- added D121: 4, LED_SMD:LED_SK6812MINI-E_3.2x2.8mm_P1.5mm_ReverseMount, symbol LED:SK6812MINI-E
- added D122: 5, LED_SMD:LED_SK6812MINI-E_3.2x2.8mm_P1.5mm_ReverseMount, symbol LED:SK6812MINI-E
- added D123: 6, LED_SMD:LED_SK6812MINI-E_3.2x2.8mm_P1.5mm_ReverseMount, symbol LED:SK6812MINI-E
- added D124: 7, LED_SMD:LED_SK6812MINI-E_3.2x2.8mm_P1.5mm_ReverseMount, symbol LED:SK6812MINI-E
- added D125: 8, LED_SMD:LED_SK6812MINI-E_3.2x2.8mm_P1.5mm_ReverseMount, symbol LED:SK6812MINI-E
- added D126: 9, LED_SMD:LED_SK6812MINI-E_3.2x2.8mm_P1.5mm_ReverseMount, symbol LED:SK6812MINI-E
- added D127: 0, LED_SMD:LED_SK6812MINI-E_3.2x2.8mm_P1.5mm_ReverseMount, symbol LED:SK6812MINI-E
- added D128: -, LED_SMD:LED_SK6812MINI-E_3.2x2.8mm_P1.5mm_ReverseMount, symbol LED:SK6812MINI-E
- added D129: =, LED_SMD:LED_SK6812MINI-E_3.2x2.8mm_P1.5mm_ReverseMount, symbol LED:SK6812MINI-E
- added D130: BSP, LED_SMD:LED_SK6812MINI-E_3.2x2.8mm_P1.5mm_ReverseMount, symbol LED:SK6812MINI-E
- added D131: INS, LED_SMD:LED_SK6812MINI-E_3.2x2.8mm_P1.5mm_ReverseMount, symbol LED:SK6812MINI-E
- added D132: HOME, LED_SMD:LED_SK6812MINI-E_3.2x2.8mm_P1.5mm_ReverseMount, symbol LED:SK6812MINI-E
- added D133, D150: PG UP, LED_SMD:LED_SK6812MINI-E_3.2x2.8mm_P1.5mm_ReverseMount, symbol LED:SK6812MINI-E
- added D134: TAB, LED_SMD:LED_SK6812MINI-E_3.2x2.8mm_P1.5mm_ReverseMount, symbol LED:SK6812MINI-E
- added D135: Q, LED_SMD:LED_SK6812MINI-E_3.2x2.8mm_P1.5mm_ReverseMount, symbol LED:SK6812MINI-E
- added D136: W, LED_SMD:LED_SK6812MINI-E_3.2x2.8mm_P1.5mm_ReverseMount, symbol LED:SK6812MINI-E
- added D137: E, LED_SMD:LED_SK6812MINI-E_3.2x2.8mm_P1.5mm_ReverseMount, symbol LED:SK6812MINI-E
- added D138: R, LED_SMD:LED_SK6812MINI-E_3.2x2.8mm_P1.5mm_ReverseMount, symbol LED:SK6812MINI-E
- added D139: T, LED_SMD:LED_SK6812MINI-E_3.2x2.8mm_P1.5mm_ReverseMount, symbol LED:SK6812MINI-E
- added D140: Y, LED_SMD:LED_SK6812MINI-E_3.2x2.8mm_P1.5mm_ReverseMount, symbol LED:SK6812MINI-E
- added D141: U, LED_SMD:LED_SK6812MINI-E_3.2x2.8mm_P1.5mm_ReverseMount, symbol LED:SK6812MINI-E
- added D142: I, LED_SMD:LED_SK6812MINI-E_3.2x2.8mm_P1.5mm_ReverseMount, symbol LED:SK6812MINI-E
- added D143: O, LED_SMD:LED_SK6812MINI-E_3.2x2.8mm_P1.5mm_ReverseMount, symbol LED:SK6812MINI-E
- added D144: P, LED_SMD:LED_SK6812MINI-E_3.2x2.8mm_P1.5mm_ReverseMount, symbol LED:SK6812MINI-E
- added D145: [, LED_SMD:LED_SK6812MINI-E_3.2x2.8mm_P1.5mm_ReverseMount, symbol LED:SK6812MINI-E
- added D146: ], LED_SMD:LED_SK6812MINI-E_3.2x2.8mm_P1.5mm_ReverseMount, symbol LED:SK6812MINI-E
- added D147: \, LED_SMD:LED_SK6812MINI-E_3.2x2.8mm_P1.5mm_ReverseMount, symbol LED:SK6812MINI-E
- added D148: DEL, LED_SMD:LED_SK6812MINI-E_3.2x2.8mm_P1.5mm_ReverseMount, symbol LED:SK6812MINI-E
- added D149: END, LED_SMD:LED_SK6812MINI-E_3.2x2.8mm_P1.5mm_ReverseMount, symbol LED:SK6812MINI-E
- added D151: CAPS, LED_SMD:LED_SK6812MINI-E_3.2x2.8mm_P1.5mm_ReverseMount, symbol LED:SK6812MINI-E
- added D152: A, LED_SMD:LED_SK6812MINI-E_3.2x2.8mm_P1.5mm_ReverseMount, symbol LED:SK6812MINI-E
- added D153: S, LED_SMD:LED_SK6812MINI-E_3.2x2.8mm_P1.5mm_ReverseMount, symbol LED:SK6812MINI-E
- added D154: D, LED_SMD:LED_SK6812MINI-E_3.2x2.8mm_P1.5mm_ReverseMount, symbol LED:SK6812MINI-E
- added D155: F, LED_SMD:LED_SK6812MINI-E_3.2x2.8mm_P1.5mm_ReverseMount, symbol LED:SK6812MINI-E
- added D156: G, LED_SMD:LED_SK6812MINI-E_3.2x2.8mm_P1.5mm_ReverseMount, symbol LED:SK6812MINI-E
- added D157: H, LED_SMD:LED_SK6812MINI-E_3.2x2.8mm_P1.5mm_ReverseMount, symbol LED:SK6812MINI-E
- added D158: J, LED_SMD:LED_SK6812MINI-E_3.2x2.8mm_P1.5mm_ReverseMount, symbol LED:SK6812MINI-E
- added D159: K, LED_SMD:LED_SK6812MINI-E_3.2x2.8mm_P1.5mm_ReverseMount, symbol LED:SK6812MINI-E
- added D160: L, LED_SMD:LED_SK6812MINI-E_3.2x2.8mm_P1.5mm_ReverseMount, symbol LED:SK6812MINI-E
- added D161: ;, LED_SMD:LED_SK6812MINI-E_3.2x2.8mm_P1.5mm_ReverseMount, symbol LED:SK6812MINI-E
- added D162: ', LED_SMD:LED_SK6812MINI-E_3.2x2.8mm_P1.5mm_ReverseMount, symbol LED:SK6812MINI-E
- added D163: ENTER, LED_SMD:LED_SK6812MINI-E_3.2x2.8mm_P1.5mm_ReverseMount, symbol LED:SK6812MINI-E
- added D164: LSHIFT, LED_SMD:LED_SK6812MINI-E_3.2x2.8mm_P1.5mm_ReverseMount, symbol LED:SK6812MINI-E
- added D165: Z, LED_SMD:LED_SK6812MINI-E_3.2x2.8mm_P1.5mm_ReverseMount, symbol LED:SK6812MINI-E
- added D166: X, LED_SMD:LED_SK6812MINI-E_3.2x2.8mm_P1.5mm_ReverseMount, symbol LED:SK6812MINI-E
- added D167: C, LED_SMD:LED_SK6812MINI-E_3.2x2.8mm_P1.5mm_ReverseMount, symbol LED:SK6812MINI-E
- added D168: V, LED_SMD:LED_SK6812MINI-E_3.2x2.8mm_P1.5mm_ReverseMount, symbol LED:SK6812MINI-E
- added D169: B, LED_SMD:LED_SK6812MINI-E_3.2x2.8mm_P1.5mm_ReverseMount, symbol LED:SK6812MINI-E
- added D170: N, LED_SMD:LED_SK6812MINI-E_3.2x2.8mm_P1.5mm_ReverseMount, symbol LED:SK6812MINI-E
- added D171: M, LED_SMD:LED_SK6812MINI-E_3.2x2.8mm_P1.5mm_ReverseMount, symbol LED:SK6812MINI-E
- added D172: ,, LED_SMD:LED_SK6812MINI-E_3.2x2.8mm_P1.5mm_ReverseMount, symbol LED:SK6812MINI-E
- added D173: ., LED_SMD:LED_SK6812MINI-E_3.2x2.8mm_P1.5mm_ReverseMount, symbol LED:SK6812MINI-E
- added D174: ?/, LED_SMD:LED_SK6812MINI-E_3.2x2.8mm_P1.5mm_ReverseMount, symbol LED:SK6812MINI-E
- added D175: RSHIFT, LED_SMD:LED_SK6812MINI-E_3.2x2.8mm_P1.5mm_ReverseMount, symbol LED:SK6812MINI-E
- added D176: UP, LED_SMD:LED_SK6812MINI-E_3.2x2.8mm_P1.5mm_ReverseMount, symbol LED:SK6812MINI-E
- added D177: LCTRL, LED_SMD:LED_SK6812MINI-E_3.2x2.8mm_P1.5mm_ReverseMount, symbol LED:SK6812MINI-E
- added D178: OS, LED_SMD:LED_SK6812MINI-E_3.2x2.8mm_P1.5mm_ReverseMount, symbol LED:SK6812MINI-E
- added D179: LALT, LED_SMD:LED_SK6812MINI-E_3.2x2.8mm_P1.5mm_ReverseMount, symbol LED:SK6812MINI-E
- added D180: SPACE, LED_SMD:LED_SK6812MINI-E_3.2x2.8mm_P1.5mm_ReverseMount, symbol LED:SK6812MINI-E
- added D181: RALT, LED_SMD:LED_SK6812MINI-E_3.2x2.8mm_P1.5mm_ReverseMount, symbol LED:SK6812MINI-E
- added D182: ANY, LED_SMD:LED_SK6812MINI-E_3.2x2.8mm_P1.5mm_ReverseMount, symbol LED:SK6812MINI-E
- added D183: MENU, LED_SMD:LED_SK6812MINI-E_3.2x2.8mm_P1.5mm_ReverseMount, symbol LED:SK6812MINI-E
- added D184: RCTRL, LED_SMD:LED_SK6812MINI-E_3.2x2.8mm_P1.5mm_ReverseMount, symbol LED:SK6812MINI-E
- added D185: LEFT, LED_SMD:LED_SK6812MINI-E_3.2x2.8mm_P1.5mm_ReverseMount, symbol LED:SK6812MINI-E
- added D186: DOWN, LED_SMD:LED_SK6812MINI-E_3.2x2.8mm_P1.5mm_ReverseMount, symbol LED:SK6812MINI-E
- added D187: RIGHT, LED_SMD:LED_SK6812MINI-E_3.2x2.8mm_P1.5mm_ReverseMount, symbol LED:SK6812MINI-E
- added J2: USB_C_Receptacle_USB2.0_14P, Connector_USB:USB_C_Receptacle_Amphenol_12401948E412A, symbol Connector:USB_C_Receptacle_USB2.0_14P
- added L1: 47uH, Inductor_SMD:L_APV_ANR3015, symbol Device:L
- added Q1: Si1308EDL, Package_TO_SOT_SMD:SOT-323_SC-70, symbol Transistor_FET:Si1308EDL
- added R1: 2.2, Resistor_SMD:R_0805_2012Metric_Pad1.20x1.40mm_HandSolder, symbol Device:R
- added R2: 1M, Resistor_SMD:R_0805_2012Metric_Pad1.20x1.40mm_HandSolder, symbol Device:R
- added R3: 1K, Resistor_SMD:R_0805_2012Metric_Pad1.20x1.40mm_HandSolder, symbol Device:R
- added R4: R, Resistor_SMD:R_0805_2012Metric_Pad1.20x1.40mm_HandSolder, symbol Device:R
- added R5, R6: 5.1K, Resistor_SMD:R_0805_2012Metric_Pad1.20x1.40mm_HandSolder, symbol Device:R_Small
- added SW1, SW100: SW_Push, Button_Switch_SMD:SW_Push_SPST_NO_Alps_SKRK, symbol Switch:SW_Push
- added SW10: F8, 1u_switch:SW_Cherry_MX_1.00u_PCB, symbol Switch:SW_Push_45deg
- added SW11: F9, 1u_switch:SW_Cherry_MX_1.00u_PCB, symbol Switch:SW_Push_45deg
- added SW12: F10, 1u_switch:SW_Cherry_MX_1.00u_PCB, symbol Switch:SW_Push_45deg
- added SW13: F11, 1u_switch:SW_Cherry_MX_1.00u_PCB, symbol Switch:SW_Push_45deg
- added SW14: F12, 1u_switch:SW_Cherry_MX_1.00u_PCB, symbol Switch:SW_Push_45deg
- added SW15: `, 1u_switch:SW_Cherry_MX_1.00u_PCB, symbol Switch:SW_Push_45deg
- added SW16: 1, 1u_switch:SW_Cherry_MX_1.00u_PCB, symbol Switch:SW_Push_45deg
- added SW17: 2, 1u_switch:SW_Cherry_MX_1.00u_PCB, symbol Switch:SW_Push_45deg
- added SW18: 3, 1u_switch:SW_Cherry_MX_1.00u_PCB, symbol Switch:SW_Push_45deg
- added SW19: 4, 1u_switch:SW_Cherry_MX_1.00u_PCB, symbol Switch:SW_Push_45deg
- added SW2: ESC, 1u_switch:SW_Cherry_MX_1.00u_PCB, symbol Switch:SW_Push_45deg
- added SW20: 5, 1u_switch:SW_Cherry_MX_1.00u_PCB, symbol Switch:SW_Push_45deg
- added SW21: 6, 1u_switch:SW_Cherry_MX_1.00u_PCB, symbol Switch:SW_Push_45deg
- added SW22: 7, 1u_switch:SW_Cherry_MX_1.00u_PCB, symbol Switch:SW_Push_45deg
- added SW23: 8, 1u_switch:SW_Cherry_MX_1.00u_PCB, symbol Switch:SW_Push_45deg
- added SW24: 9, 1u_switch:SW_Cherry_MX_1.00u_PCB, symbol Switch:SW_Push_45deg
- added SW25: 0, 1u_switch:SW_Cherry_MX_1.00u_PCB, symbol Switch:SW_Push_45deg
- added SW26: -, 1u_switch:SW_Cherry_MX_1.00u_PCB, symbol Switch:SW_Push_45deg
- added SW27: =, 1u_switch:SW_Cherry_MX_1.00u_PCB, symbol Switch:SW_Push_45deg
- added SW28: BACKSPACE, Button_Switch_Keyboard:SW_Cherry_MX_2.00u_PCB, symbol Switch:SW_Push_45deg
- added SW29: TAB, Button_Switch_Keyboard:SW_Cherry_MX_1.50u_PCB, symbol Switch:SW_Push_45deg
- added SW3: F1, 1u_switch:SW_Cherry_MX_1.00u_PCB, symbol Switch:SW_Push_45deg
- added SW30: Q, 1u_switch:SW_Cherry_MX_1.00u_PCB, symbol Switch:SW_Push_45deg
- added SW31: W, 1u_switch:SW_Cherry_MX_1.00u_PCB, symbol Switch:SW_Push_45deg
- added SW32: E, 1u_switch:SW_Cherry_MX_1.00u_PCB, symbol Switch:SW_Push_45deg
- added SW33: R, 1u_switch:SW_Cherry_MX_1.00u_PCB, symbol Switch:SW_Push_45deg
- added SW34: T, 1u_switch:SW_Cherry_MX_1.00u_PCB, symbol Switch:SW_Push_45deg
- added SW35: Y, 1u_switch:SW_Cherry_MX_1.00u_PCB, symbol Switch:SW_Push_45deg
- added SW36: U, 1u_switch:SW_Cherry_MX_1.00u_PCB, symbol Switch:SW_Push_45deg
- added SW37: I, 1u_switch:SW_Cherry_MX_1.00u_PCB, symbol Switch:SW_Push_45deg
- added SW38: O, 1u_switch:SW_Cherry_MX_1.00u_PCB, symbol Switch:SW_Push_45deg
- added SW39: P, 1u_switch:SW_Cherry_MX_1.00u_PCB, symbol Switch:SW_Push_45deg
- added SW4: F2, 1u_switch:SW_Cherry_MX_1.00u_PCB, symbol Switch:SW_Push_45deg
- added SW40: [, 1u_switch:SW_Cherry_MX_1.00u_PCB, symbol Switch:SW_Push_45deg
- added SW41: ], 1u_switch:SW_Cherry_MX_1.00u_PCB, symbol Switch:SW_Push_45deg
- added SW42: \, Button_Switch_Keyboard:SW_Cherry_MX_1.50u_PCB, symbol Switch:SW_Push_45deg
- added SW43: CAPS, Button_Switch_Keyboard:SW_Cherry_MX_1.75u_PCB, symbol Switch:SW_Push_45deg
- added SW44: A, 1u_switch:SW_Cherry_MX_1.00u_PCB, symbol Switch:SW_Push_45deg
- added SW45: S, 1u_switch:SW_Cherry_MX_1.00u_PCB, symbol Switch:SW_Push_45deg
- added SW46: D, 1u_switch:SW_Cherry_MX_1.00u_PCB, symbol Switch:SW_Push_45deg
- added SW47: F, 1u_switch:SW_Cherry_MX_1.00u_PCB, symbol Switch:SW_Push_45deg
- added SW48: G, 1u_switch:SW_Cherry_MX_1.00u_PCB, symbol Switch:SW_Push_45deg
- added SW49: H, 1u_switch:SW_Cherry_MX_1.00u_PCB, symbol Switch:SW_Push_45deg
- added SW5: F3, 1u_switch:SW_Cherry_MX_1.00u_PCB, symbol Switch:SW_Push_45deg
- added SW50: J, 1u_switch:SW_Cherry_MX_1.00u_PCB, symbol Switch:SW_Push_45deg
- added SW51: K, 1u_switch:SW_Cherry_MX_1.00u_PCB, symbol Switch:SW_Push_45deg
- added SW52: L, 1u_switch:SW_Cherry_MX_1.00u_PCB, symbol Switch:SW_Push_45deg
- added SW53: ;, 1u_switch:SW_Cherry_MX_1.00u_PCB, symbol Switch:SW_Push_45deg
- added SW54: ', 1u_switch:SW_Cherry_MX_1.00u_PCB, symbol Switch:SW_Push_45deg
- added SW55: ENTER, Button_Switch_Keyboard:SW_Cherry_MX_2.25u_PCB, symbol Switch:SW_Push_45deg
- added SW56: LSHIFT, Button_Switch_Keyboard:SW_Cherry_MX_2.25u_PCB, symbol Switch:SW_Push_45deg
- added SW57: Z, 1u_switch:SW_Cherry_MX_1.00u_PCB, symbol Switch:SW_Push_45deg
- added SW58: X, 1u_switch:SW_Cherry_MX_1.00u_PCB, symbol Switch:SW_Push_45deg
- added SW59: C, 1u_switch:SW_Cherry_MX_1.00u_PCB, symbol Switch:SW_Push_45deg
- added SW6: F4, 1u_switch:SW_Cherry_MX_1.00u_PCB, symbol Switch:SW_Push_45deg
- added SW60: V, 1u_switch:SW_Cherry_MX_1.00u_PCB, symbol Switch:SW_Push_45deg
- added SW61: B, 1u_switch:SW_Cherry_MX_1.00u_PCB, symbol Switch:SW_Push_45deg
- added SW62: N, 1u_switch:SW_Cherry_MX_1.00u_PCB, symbol Switch:SW_Push_45deg
- added SW63: M, 1u_switch:SW_Cherry_MX_1.00u_PCB, symbol Switch:SW_Push_45deg
- added SW64: ,, 1u_switch:SW_Cherry_MX_1.00u_PCB, symbol Switch:SW_Push_45deg
- added SW65: ., 1u_switch:SW_Cherry_MX_1.00u_PCB, symbol Switch:SW_Push_45deg
- added SW66: ?/, 1u_switch:SW_Cherry_MX_1.00u_PCB, symbol Switch:SW_Push_45deg
- added SW67: RSHIFT, Button_Switch_Keyboard:SW_Cherry_MX_2.75u_PCB, symbol Switch:SW_Push_45deg
- added SW68: LCTRL, Button_Switch_Keyboard:SW_Cherry_MX_1.25u_PCB, symbol Switch:SW_Push_45deg
- added SW69: OS, Button_Switch_Keyboard:SW_Cherry_MX_1.25u_PCB, symbol Switch:SW_Push_45deg
- added SW7: F5, 1u_switch:SW_Cherry_MX_1.00u_PCB, symbol Switch:SW_Push_45deg
- added SW70: LALT, Button_Switch_Keyboard:SW_Cherry_MX_1.25u_PCB, symbol Switch:SW_Push_45deg
- added SW71: SPACE, Button_Switch_Keyboard:SW_Cherry_MX_6.25u_PCB, symbol Switch:SW_Push_45deg
- added SW72: RALT, Button_Switch_Keyboard:SW_Cherry_MX_1.25u_PCB, symbol Switch:SW_Push_45deg
- added SW73: ANY, Button_Switch_Keyboard:SW_Cherry_MX_1.25u_PCB, symbol Switch:SW_Push_45deg
- added SW74: MENU, Button_Switch_Keyboard:SW_Cherry_MX_1.25u_PCB, symbol Switch:SW_Push_45deg
- added SW75: RCTRL, Button_Switch_Keyboard:SW_Cherry_MX_1.25u_PCB, symbol Switch:SW_Push_45deg
- added SW76: PRINT, Button_Switch_Keyboard:SW_Cherry_MX_1.00u_PCB, symbol Switch:SW_Push_45deg
- added SW77: PAUSE, 1u_switch:SW_Cherry_MX_1.00u_PCB, symbol Switch:SW_Push_45deg
- added SW78: SCR LOCK, 1u_switch:SW_Cherry_MX_1.00u_PCB, symbol Switch:SW_Push_45deg
- added SW79: INS, 1u_switch:SW_Cherry_MX_1.00u_PCB, symbol Switch:SW_Push_45deg
- added SW8: F6, 1u_switch:SW_Cherry_MX_1.00u_PCB, symbol Switch:SW_Push_45deg
- added SW80: HM, 1u_switch:SW_Cherry_MX_1.00u_PCB, symbol Switch:SW_Push_45deg
- added SW81: PU, 1u_switch:SW_Cherry_MX_1.00u_PCB, symbol Switch:SW_Push_45deg
- added SW82: DEL, 1u_switch:SW_Cherry_MX_1.00u_PCB, symbol Switch:SW_Push_45deg
- added SW83: END, 1u_switch:SW_Cherry_MX_1.00u_PCB, symbol Switch:SW_Push_45deg
- added SW84: PD, 1u_switch:SW_Cherry_MX_1.00u_PCB, symbol Switch:SW_Push_45deg
- added SW85: LEFT, 1u_switch:SW_Cherry_MX_1.00u_PCB, symbol Switch:SW_Push_45deg
- added SW86: UP, 1u_switch:SW_Cherry_MX_1.00u_PCB, symbol Switch:SW_Push_45deg
- added SW87: RIGHT, 1u_switch:SW_Cherry_MX_1.00u_PCB, symbol Switch:SW_Push_45deg
- added SW88: DOWN, 1u_switch:SW_Cherry_MX_1.00u_PCB, symbol Switch:SW_Push_45deg
- added SW9: F7, 1u_switch:SW_Cherry_MX_1.00u_PCB, symbol Switch:SW_Push_45deg
- added U1: AP2112K-3.3, Package_TO_SOT_SMD:SOT-23-5, symbol Regulator_Linear:AP2112K-3.3
- added U2: RP2040, Package_DFN_QFN:QFN-56-1EP_7x7mm_P0.4mm_EP3.2x3.2mm, symbol MCU_RaspberryPi:RP2040
- added U3: W25Q128JVS, Package_SO:SOIC-8_5.3x5.3mm_P1.27mm, symbol Memory_Flash:W25Q128JVS
- added Y1: Crystal_GND24, Crystal:Crystal_SMD_3225-4Pin_3.2x2.5mm_HandSoldering, symbol Device:Crystal_GND24
- J1: footprint Connector_FFC-FPC:Molex_502231-2400_1x24-1SH_P0.5mm_Vertical -> Library:Molex_502231-2400_1x24-1SH_P0.5mm_Vertical
Connections:
- net RES: now reaches J1.10 (Pin_10)
- net RES: now also U2.7 (GPIO5)
- net D/C: now reaches J1.11 (Pin_11)
- net D/C: now also U2.8 (GPIO6)
- net CS: now reaches J1.12 (Pin_12)
- net CS: now also U2.9 (GPIO7)
- net SCLK: now reaches J1.13 (Pin_13)
- net SCLK: now also U2.4 (GPIO2)
- net SDI: now reaches J1.14 (Pin_14)
- net SDI: now also U2.5 (GPIO3)
- net +3V3: now reaches J1.15 (Pin_15)
- net +3V3: now also J1.16 (Pin_16), C1.1, C13.2, C16.2, C17.2, C18.2, C19.2, C20.2, C3.1, C5.1, L1.1, R4.1, U1.5 (VOUT), U2.1 (IOVDD), U2.10 (IOVDD), U2.22 (IOVDD), U2.33 (IOVDD), U2.42 (IOVDD), U2.43 (ADC_AVDD), U2.44 (VREG_VIN), U2.48 (USB_VDD), U2.49 (IOVDD), U3.8 (VCC)
- net GND: now reaches J1.17 (Pin_17)
- net GND: now also J1.8 (Pin_8), C1.2, C10.1, C11.1, C12.1, C13.1, C14.1, C15.1, C16.1, C17.1, C18.1, C19.1, C2.2, C20.1, C21.2, C22.2, C3.2, C4.1, C5.2, C7.2, C8.1, C9.1, D101.1 (VSS), D102.1 (VSS), D103.1 (VSS), D104.1 (VSS), D105.1 (VSS), D106.1 (VSS), D107.1 (VSS), D108.1 (VSS), D109.1 (VSS), D110.1 (VSS), D111.1 (VSS), D112.1 (VSS), D113.1 (VSS), D114.1 (VSS), D115.1 (VSS), D116.1 (VSS), D117.1 (VSS), D118.1 (VSS), D119.1 (VSS), D120.1 (VSS), D121.1 (VSS), D122.1 (VSS), D123.1 (VSS), D124.1 (VSS), D125.1 (VSS), D126.1 (VSS), D127.1 (VSS), D128.1 (VSS), D129.1 (VSS), D130.1 (VSS), D131.1 (VSS), D132.1 (VSS), D133.1 (VSS), D134.1 (VSS), D135.1 (VSS), D136.1 (VSS), D137.1 (VSS), D138.1 (VSS), D139.1 (VSS), D140.1 (VSS), D141.1 (VSS), D142.1 (VSS), D143.1 (VSS), D144.1 (VSS), D145.1 (VSS), D146.1 (VSS), D147.1 (VSS), D148.1 (VSS), D149.1 (VSS), D150.1 (VSS), D151.1 (VSS), D152.1 (VSS), D153.1 (VSS), D154.1 (VSS), D155.1 (VSS), D156.1 (VSS), D157.1 (VSS), D158.1 (VSS), D159.1 (VSS), D160.1 (VSS), D161.1 (VSS), D162.1 (VSS), D163.1 (VSS), D164.1 (VSS), D165.1 (VSS), D166.1 (VSS), D167.1 (VSS), D168.1 (VSS), D169.1 (VSS), D170.1 (VSS), D171.1 (VSS), D172.1 (VSS), D173.1 (VSS), D174.1 (VSS), D175.1 (VSS), D176.1 (VSS), D177.1 (VSS), D178.1 (VSS), D179.1 (VSS), D180.1 (VSS), D181.1 (VSS), D182.1 (VSS), D183.1 (VSS), D184.1 (VSS), D185.1 (VSS), D186.1 (VSS), D187.1 (VSS), D99.1 (K), J2.A1 (GND), J2.A12 (GND), J2.B1 (GND), J2.B12 (GND), J2.SH (SHIELD), R1.2, R2.2, R5.2, R6.2, SW1.1, SW100.1, U1.2 (GND), U2.19 (TESTEN), U2.57 (GND), U3.4 (GND), Y1.2 (G), Y1.4 (G)
- net at J1.18 (Pin_18): now also C8.2
- net GDR: now reaches J1.2 (Pin_2)
- net GDR: now also Q1.1 (G), R2.1
- net at J1.20 (Pin_20): now also C9.2
- net VGH: now reaches J1.21 (Pin_21)
- net VGH: now also C7.1, D100.1 (K)
- net at J1.22 (Pin_22): now also C10.2
- net VGL: now reaches J1.23 (Pin_23)
- net VGL: now also C11.2, D98.2 (A)
- net at J1.24 (Pin_24): now also C12.2
- net RESE: now reaches J1.3 (Pin_3)
- net RESE: now also Q1.2 (S), R1.1
- net at J1.5 (Pin_5): now also C4.2
- net BUSY: now reaches J1.9 (Pin_9)
- net BUSY: now also U2.6 (GPIO4)
- new net: D179.4 (DOUT), D180.2 (DIN)
- new net: D180.4 (DOUT), D181.2 (DIN)
- new net: C6.2, D100.2 (A), L1.2, Q1.3 (D)
- new net: D133.4 (DOUT), D134.2 (DIN)
- new net: D134.4 (DOUT), D135.2 (DIN)
- new net: D17.2 (A), SW15.2
- new net: D19.2 (A), SW17.2
- new net: D11.2 (A), SW12.2
- new net: D22.2 (A), SW20.2
- new net: D36.2 (A), SW31.2
- new net: D131.4 (DOUT), D132.2 (DIN)
- new net: D132.4 (DOUT), D133.2 (DIN)
- new net: D2.2 (A), SW3.2
- new net: D30.2 (A), SW28.2
- new net: D59.2 (A), SW51.2
- new net: D52.2 (A), SW44.2
- new net: D70.2 (A), SW62.2
- new net: D8.2 (A), SW9.2
- new net: D50.2 (A), SW84.2
- new net: D81.2 (A), SW72.2
- new net: D13.2 (A), SW14.2
- new net: D29.2 (A), SW27.2
- new net: D63.2 (A), SW55.2
- new net: D16.2 (A), SW78.2
- new net: D147.4 (DOUT), D148.2 (DIN)
- new net: D148.4 (DOUT), D149.2 (DIN)
- new net: D121.4 (DOUT), D122.2 (DIN)
- new net: D122.4 (DOUT), D123.2 (DIN)
- new net: D25.2 (A), SW23.2
- new net: D105.4 (DOUT), D106.2 (DIN)
- new net: D106.4 (DOUT), D107.2 (DIN)
- new net: D78.2 (A), SW69.2
- new net: D84.2 (A), SW75.2
- new net: D185.4 (DOUT), D186.2 (DIN)
- new net: D186.4 (DOUT), D187.2 (DIN)
- new net: D55.2 (A), SW47.2
- new net: D80.2 (A), SW71.2
- new net: D114.4 (DOUT), D115.2 (DIN)
- new net: D115.4 (DOUT), D116.2 (DIN)
- new net: D51.2 (A), SW43.2
- new net: D61.2 (A), SW53.2
- new net: C6.1, D98.1 (K), D99.2 (A)
- new net: D54.2 (A), SW46.2
- new net: D34.2 (A), SW29.2
- new net: D126.4 (DOUT), D127.2 (DIN)
- new net: D127.4 (DOUT), D128.2 (DIN)
- new net: D4.2 (A), SW5.2
- new net: D64.2 (A), SW56.2
- new net: D111.4 (DOUT), D112.2 (DIN)
- new net: D112.4 (DOUT), D113.2 (DIN)
- new net: D123.4 (DOUT), D124.2 (DIN)
- new net: D107.4 (DOUT), D108.2 (DIN)
- new net: D26.2 (A), SW24.2
- new net: D38.2 (A), SW33.2
- new net: D66.2 (A), SW58.2
- new net: D42.2 (A), SW37.2
- new net: D48.2 (A), SW82.2
- new net: D68.2 (A), SW60.2
- new net: D151.4 (DOUT), D152.2 (DIN)
- new net: D152.4 (DOUT), D153.2 (DIN)
- new net: D117.4 (DOUT), D118.2 (DIN)
- new net: D118.4 (DOUT), D119.2 (DIN)
- new net: D163.4 (DOUT), D164.2 (DIN)
- new net: D164.4 (DOUT), D165.2 (DIN)
- new net: D160.4 (DOUT), D161.2 (DIN)
- new net: D161.4 (DOUT), D162.2 (DIN)
- new net: D113.4 (DOUT), D114.2 (DIN)
- new net: D125.4 (DOUT), D126.2 (DIN)
- new net: D86.2 (A), SW88.2
- new net: D3.2 (A), SW4.2
- new net: D173.4 (DOUT), D174.2 (DIN)
- new net: D174.4 (DOUT), D175.2 (DIN)
- new net: D10.2 (A), SW11.2
- new net: D143.4 (DOUT), D144.2 (DIN)
- new net: D144.4 (DOUT), D145.2 (DIN)
- new net: D47.2 (A), SW42.2
- new net: D176.4 (DOUT), D177.2 (DIN)
- new net: D177.4 (DOUT), D178.2 (DIN)
- new net: D139.4 (DOUT), D140.2 (DIN)
- new net: D140.4 (DOUT), D141.2 (DIN)
- new net: D75.2 (A), SW67.2
- new net: D74.2 (A), SW66.2
- new net: D58.2 (A), SW50.2
- new net: D41.2 (A), SW36.2
- new net: D169.4 (DOUT), D170.2 (DIN)
- new net: D170.4 (DOUT), D171.2 (DIN)
- new net: D77.2 (A), SW68.2
- new net: D45.2 (A), SW40.2
- new net: D154.4 (DOUT), D155.2 (DIN)
- new net: D155.4 (DOUT), D156.2 (DIN)
- new net: D71.2 (A), SW63.2
- new net: D67.2 (A), SW59.2
- new net: D157.4 (DOUT), D158.2 (DIN)
- new net: D158.4 (DOUT), D159.2 (DIN)
- new net: D44.2 (A), SW39.2
- new net: D171.4 (DOUT), D172.2 (DIN)
- new net: D31.2 (A), SW79.2
- new net: D181.4 (DOUT), D182.2 (DIN)
- new net: D182.4 (DOUT), D183.2 (DIN)
- new net: D57.2 (A), SW49.2
- new net: D21.2 (A), SW19.2
- new net: D104.4 (DOUT), D105.2 (DIN)
- new net: D39.2 (A), SW34.2
- new net: D73.2 (A), SW65.2
- new net: R3.1, SW1.2
- new net: D178.4 (DOUT), D179.2 (DIN)
- new net: D5.2 (A), SW6.2
- new net: D130.4 (DOUT), D131.2 (DIN)
- new net: D82.2 (A), SW73.2
- new net: D175.4 (DOUT), D176.2 (DIN)
- new net: D53.2 (A), SW45.2
- new net: D145.4 (DOUT), D146.2 (DIN)
- new net: D146.4 (DOUT), D147.2 (DIN)
- new net: D24.2 (A), SW22.2
- new net: D12.2 (A), SW13.2
- new net: D72.2 (A), SW64.2
- new net: D35.2 (A), SW30.2
- new net: D15.2 (A), SW77.2
- new net: D165.4 (DOUT), D166.2 (DIN)
- new net: D166.4 (DOUT), D167.2 (DIN)
- new net: D136.4 (DOUT), D137.2 (DIN)
- new net: D137.4 (DOUT), D138.2 (DIN)
- new net: D83.2 (A), SW74.2
- new net: D43.2 (A), SW38.2
- new net: D20.2 (A), SW18.2
- new net: D76.2 (A), SW86.2
- new net: D141.4 (DOUT), D142.2 (DIN)
- new net: D142.4 (DOUT), D143.2 (DIN)
- new net: D109.4 (DOUT), D110.2 (DIN)
- new net: D110.4 (DOUT), D111.2 (DIN)
- new net: D87.2 (A), SW87.2
- new net: D18.2 (A), SW16.2
- new net: D37.2 (A), SW32.2
- new net: D62.2 (A), SW54.2
- new net: D28.2 (A), SW26.2
- new net: D49.2 (A), SW83.2
- new net: R4.2, SW100.2, U2.26 (RUN)
- new net: D40.2 (A), SW35.2
- new net: D102.4 (DOUT), D103.2 (DIN)
- new net: D103.4 (DOUT), D104.2 (DIN)
- new net: D167.4 (DOUT), D168.2 (DIN)
- new net: D168.4 (DOUT), D169.2 (DIN)
- new net: D101.4 (DOUT), D102.2 (DIN)
- new net: D159.4 (DOUT), D160.2 (DIN)
- new net: D23.2 (A), SW21.2
- new net: J2.A5 (CC1), R5.1
- new net: J2.B5 (CC2), R6.1
- new net: D183.4 (DOUT), D184.2 (DIN)
- new net: D184.4 (DOUT), D185.2 (DIN)
- new net: D149.4 (DOUT), D150.2 (DIN)
- new net: D56.2 (A), SW48.2
- new net: D116.4 (DOUT), D117.2 (DIN)
- new net: D69.2 (A), SW61.2
- new net: D128.4 (DOUT), D129.2 (DIN)
- new net: D129.4 (DOUT), D130.2 (DIN)
- new net: D46.2 (A), SW41.2
- new net: D1.2 (A), SW2.2
- new net: D156.4 (DOUT), D157.2 (DIN)
- new net: D120.4 (DOUT), D121.2 (DIN)
- new net: D172.4 (DOUT), D173.2 (DIN)
- new net: D9.2 (A), SW10.2
- new net: D33.2 (A), SW81.2
- new net: D7.2 (A), SW8.2
- new net: D124.4 (DOUT), D125.2 (DIN)
- new net: D65.2 (A), SW57.2
- new net: D32.2 (A), SW80.2
- new net: D27.2 (A), SW25.2
- new net: D153.4 (DOUT), D154.2 (DIN)
- new net: D60.2 (A), SW52.2
- new net: D6.2 (A), SW7.2
- new net: D85.2 (A), SW85.2
- new net: D135.4 (DOUT), D136.2 (DIN)
- new net: D108.4 (DOUT), D109.2 (DIN)
- new net: D14.2 (A), SW76.2
- new net: D138.4 (DOUT), D139.2 (DIN)
- new net: D150.4 (DOUT), D151.2 (DIN)
- new net: D119.4 (DOUT), D120.2 (DIN)
- new net: D162.4 (DOUT), D163.2 (DIN)
- new net: D79.2 (A), SW70.2
- new net +1V1: C14.2, C15.2, U2.23 (DVDD), U2.45 (VREG_VOUT), U2.50 (DVDD)
- new net COL0: SW15.1, SW2.1, SW29.1, SW43.1, SW56.1, SW68.1, U2.36 (GPIO24)
- new net COL1: SW16.1, SW30.1, SW44.1, SW69.1, U2.35 (GPIO23)
- new net COL10: SW11.1, SW25.1, SW39.1, SW53.1, SW65.1, SW72.1, U2.17 (GPIO14)
- new net COL11: SW12.1, SW26.1, SW40.1, SW54.1, SW66.1, SW73.1, U2.16 (GPIO13)
- new net COL12: SW13.1, SW27.1, SW41.1, SW74.1, U2.15 (GPIO12)
- new net COL13: SW14.1, SW28.1, SW42.1, SW55.1, SW67.1, SW75.1, U2.14 (GPIO11)
- new net COL14: SW76.1, SW79.1, SW82.1, SW85.1, U2.13 (GPIO10)
- new net COL15: SW77.1, SW80.1, SW83.1, SW86.1, SW88.1, U2.12 (GPIO9)
- new net COL16: SW78.1, SW81.1, SW84.1, SW87.1, U2.11 (GPIO8)
- new net COL2: SW17.1, SW3.1, SW31.1, SW45.1, SW57.1, SW70.1, U2.34 (GPIO22)
- new net COL3: SW18.1, SW32.1, SW4.1, SW46.1, SW58.1, U2.32 (GPIO21)
- new net COL4: SW19.1, SW33.1, SW47.1, SW5.1, SW59.1, U2.31 (GPIO20)
- new net COL5: SW20.1, SW34.1, SW48.1, SW6.1, SW60.1, U2.30 (GPIO19)
- new net COL6: SW21.1, SW35.1, SW49.1, SW61.1, SW7.1, U2.29 (GPIO18)
- new net COL7: SW22.1, SW36.1, SW50.1, SW62.1, SW71.1, SW8.1, U2.28 (GPIO17)
- new net COL8: SW23.1, SW37.1, SW51.1, SW63.1, SW9.1, U2.27 (GPIO16)
- new net COL9: SW10.1, SW24.1, SW38.1, SW52.1, SW64.1, U2.18 (GPIO15)
- new net F_CLK: U2.52 (QSPI_SCLK), U3.6 (CLK)
- new net F_CS: R3.2, U2.56 (~{QSPI_SS}), U3.1 (~{CS})
- new net F_SD0: U2.53 (QSPI_SD0), U3.5 (DI/IO_{0})
- new net F_SD1: U2.55 (QSPI_SD1), U3.2 (DO/IO_{1})
- new net F_SD2: U2.54 (QSPI_SD2), U3.3 (~{WP}/IO_{2})
- new net F_SD3: U2.51 (QSPI_SD3), U3.7 (~{HOLD}/~{RESET}/IO_{3})
- new net LED_DIN: D101.2 (DIN), U2.3 (GPIO1)
- new net ROW0: D1.1 (K), D10.1 (K), D11.1 (K), D12.1 (K), D13.1 (K), D14.1 (K), D15.1 (K), D16.1 (K), D2.1 (K), D3.1 (K), D4.1 (K), D5.1 (K), D6.1 (K), D7.1 (K), D8.1 (K), D9.1 (K), U2.2 (GPIO0)
- new net ROW1: D17.1 (K), D18.1 (K), D19.1 (K), D20.1 (K), D21.1 (K), D22.1 (K), D23.1 (K), D24.1 (K), D25.1 (K), D26.1 (K), D27.1 (K), D28.1 (K), D29.1 (K), D30.1 (K), D31.1 (K), D32.1 (K), D33.1 (K), U2.41 (GPIO29/ADC3)
- new net ROW2: D34.1 (K), D35.1 (K), D36.1 (K), D37.1 (K), D38.1 (K), D39.1 (K), D40.1 (K), D41.1 (K), D42.1 (K), D43.1 (K), D44.1 (K), D45.1 (K), D46.1 (K), D47.1 (K), D48.1 (K), D49.1 (K), D50.1 (K), U2.40 (GPIO28/ADC2)
- new net ROW3: D51.1 (K), D52.1 (K), D53.1 (K), D54.1 (K), D55.1 (K), D56.1 (K), D57.1 (K), D58.1 (K), D59.1 (K), D60.1 (K), D61.1 (K), D62.1 (K), D63.1 (K), U2.39 (GPIO27/ADC1)
- new net ROW4: D64.1 (K), D65.1 (K), D66.1 (K), D67.1 (K), D68.1 (K), D69.1 (K), D70.1 (K), D71.1 (K), D72.1 (K), D73.1 (K), D74.1 (K), D75.1 (K), D76.1 (K), U2.38 (GPIO26/ADC0)
- new net ROW5: D77.1 (K), D78.1 (K), D79.1 (K), D80.1 (K), D81.1 (K), D82.1 (K), D83.1 (K), D84.1 (K), D85.1 (K), D86.1 (K), D87.1 (K), U2.37 (GPIO25)
- new net USB_D+: J2.A6 (D+), J2.B6 (D+), U2.47 (USB_DP)
- new net USB_D-: J2.A7 (D-), J2.B7 (D-), U2.46 (USB_DM)
- new net VBUS: C2.1, D101.3 (VDD), D102.3 (VDD), D103.3 (VDD), D104.3 (VDD), D105.3 (VDD), D106.3 (VDD), D107.3 (VDD), D108.3 (VDD), D109.3 (VDD), D110.3 (VDD), D111.3 (VDD), D112.3 (VDD), D113.3 (VDD), D114.3 (VDD), D115.3 (VDD), D116.3 (VDD), D117.3 (VDD), D118.3 (VDD), D119.3 (VDD), D120.3 (VDD), D121.3 (VDD), D122.3 (VDD), D123.3 (VDD), D124.3 (VDD), D125.3 (VDD), D126.3 (VDD), D127.3 (VDD), D128.3 (VDD), D129.3 (VDD), D130.3 (VDD), D131.3 (VDD), D132.3 (VDD), D133.3 (VDD), D134.3 (VDD), D135.3 (VDD), D136.3 (VDD), D137.3 (VDD), D138.3 (VDD), D139.3 (VDD), D140.3 (VDD), D141.3 (VDD), D142.3 (VDD), D143.3 (VDD), D144.3 (VDD), D145.3 (VDD), D146.3 (VDD), D147.3 (VDD), D148.3 (VDD), D149.3 (VDD), D150.3 (VDD), D151.3 (VDD), D152.3 (VDD), D153.3 (VDD), D154.3 (VDD), D155.3 (VDD), D156.3 (VDD), D157.3 (VDD), D158.3 (VDD), D159.3 (VDD), D160.3 (VDD), D161.3 (VDD), D162.3 (VDD), D163.3 (VDD), D164.3 (VDD), D165.3 (VDD), D166.3 (VDD), D167.3 (VDD), D168.3 (VDD), D169.3 (VDD), D170.3 (VDD), D171.3 (VDD), D172.3 (VDD), D173.3 (VDD), D174.3 (VDD), D175.3 (VDD), D176.3 (VDD), D177.3 (VDD), D178.3 (VDD), D179.3 (VDD), D180.3 (VDD), D181.3 (VDD), D182.3 (VDD), D183.3 (VDD), D184.3 (VDD), D185.3 (VDD), D186.3 (VDD), D187.3 (VDD), J2.A4 (VBUS), J2.A9 (VBUS), J2.B4 (VBUS), J2.B9 (VBUS), U1.1 (VIN), U1.3 (EN)
- new net XIN: C22.1, U2.20 (XIN), Y1.1
- new net XOUT: C21.1, U2.21 (XOUT), Y1.3
- no-connect marks 0 -> 9
Other:
- note added: "i no have debugger :-("
- note added: "temp sensor optional"
- moved on the sheet: J1
